File: Hardware/Right Split Keyboard.kicad_sch (KiCad schematic)
At the start: 48 parts, among them CN2 1.0-2P WT, M5 MountingHole, M6 MountingHole, M7 MountingHole, SW18 Switch, SW19 Switch, SW20 Switch, SW21 Switch, SW22 Switch, SW23 Switch, SW24 EC11, SW25 Switch, SW26 Switch, SW27 Switch, SW28 Switch, SW29 Switch, SW30 Switch, SW31 Switch, SW32 Switch, SW33 Switch, SW34 Switch, U2 XIAO-nRF52840-SMD

Commit message: Plate fixes
Parts:
- removed C3, C4, C6: 10nF, Capacitor_SMD:C_0805_2012Metric, symbol Device:C
- removed R7, R8: 10k, Resistor_SMD:R_0805_2012Metric, symbol Device:R
Connections:
- net COL1: now also SW34.1
- net COL3: no longer SW34.1
- net R_Encoder_A: now also SW24.A
- net R_Encoder_B: now also SW24.B
Other:
- moved on the sheet: D32, SW24, SW34
