File: Hardware/Left Split Keyboard.kicad_pcb (KiCad board)
At the start: 2 copper layers, 96.2 x 97.9 mm, 44 parts, among them CN2 1.0-2P WT, SW18 Switch, SW19 Switch, SW20 Switch, SW21 Switch, SW22 Switch, SW23 Switch, SW24 EC11, SW25 Switch, SW26 Switch, SW27 Switch, SW28 Switch, SW29 Switch, SW30 Switch, SW31 Switch, SW32 Switch, SW33 Switch, SW34 Switch, U2 XIAO-nRF52840-SMD

Commit message: Finally Final
Parts:
- added REF**: MountingHole_2.2mm_M2, MountingHole:MountingHole_2.2mm_M2, F.Cu at (177.8, 50.0)
- added REF**: MountingHole_2.2mm_M2, MountingHole:MountingHole_2.2mm_M2, F.Cu at (150.2, 122.8)
- added REF**: MountingHole_2.2mm_M2, MountingHole:MountingHole_2.2mm_M2, F.Cu at (190.8, 141.0)
- added REF**: MountingHole_2.2mm_M2, MountingHole:MountingHole_2.2mm_M2, F.Cu at (113.2, 57.8)
- added REF**: MountingHole_2.2mm_M2, MountingHole:MountingHole_2.2mm_M2, F.Cu at (119.8, 122.8)
- added REF**: MountingHole_2.2mm_M2, MountingHole:MountingHole_2.2mm_M2, F.Cu at (190.8, 62.8)
- moved SW24 0.25 mm to (175.5, 129.5)
Routing:
- net /Right/ROW2: track 174.2 -> 178.6 mm
- net Net-(C4-Pad1): track 146.5 -> 148.6 mm
- net /Right/ROW0: track 136.6 -> 138.4 mm
- net /Right/ROW1: track 161.6 -> 163.3 mm
- net /Right/SW: track 90.9 -> 92.3 mm
- net Net-(C3-Pad2): track 125.5 -> 124.6 mm
- net /Right/ROW3: track 83.9 -> 83.1 mm
- net GND: vias 124 -> 122

Commit message: Plate fixes
Parts:
- removed C3, C4, C6: 10nF, Capacitor_SMD:C_0805_2012Metric
- removed CN2: 1.0-2P WT, lcsc:CONN-SMD_2P-P1.00_SHOU-HAN_1.0-2P-WT
- removed D17, D18, D19, D20, D21, D22, D23, D24, D25, D26, D27, D28, D29, D30, D31, D32: D, Diode_SMD:D_SOD-123
- removed R5: 806k, Resistor_SMD:R_0805_2012Metric
- removed R6: 2M, Resistor_SMD:R_0805_2012Metric
- removed R7, R8: 10k, Resistor_SMD:R_0805_2012Metric
- removed SW18, SW19, SW20, SW21, SW22, SW23, SW25, SW26, SW27, SW28, SW29, SW30, SW31, SW32, SW33, SW34: Switch, ScottoKeebs_Hotswap:Hotswap_MX_1.00u
- removed SW24: EC11, Rotary Encoders:RotaryEncoder_Alps_EC11E-Switch_Vertical_H20mm
- removed TP3: GND, TestPoint:TestPoint_Pad_D2.0mm
- removed TP4: VBAT, TestPoint:TestPoint_Pad_D2.0mm
- removed U2: XIAO-nRF52840-SMD, Fixed Footprints:XIAO-nRF52840-SMD Fixed
- added CN1: 1.0-2P WT, lcsc:CONN-SMD_2P-P1.00_SHOU-HAN_1.0-2P-WT, F.Cu at (138.3, 50.8)
- added D1: D, Diode_SMD:D_SOD-123, B.Cu at (115.9, 76.6)
- added D10: D, Diode_SMD:D_SOD-123, B.Cu at (173.1, 76.7)
- added D11: D, Diode_SMD:D_SOD-123, B.Cu at (173.0, 95.5)
- added D12: D, Diode_SMD:D_SOD-123, B.Cu at (173.0, 114.8)
- added D13: D, Diode_SMD:D_SOD-123, B.Cu at (192.0, 114.8)
- added D14: D, Diode_SMD:D_SOD-123, B.Cu at (191.9, 76.7)
- added D15: D, Diode_SMD:D_SOD-123, B.Cu at (192.0, 95.7)
- added D16: D, Diode_SMD:D_SOD-123, B.Cu at (173.0, 133.8)
- added D2: D, Diode_SMD:D_SOD-123, B.Cu at (116.0, 95.7)
- added D3: D, Diode_SMD:D_SOD-123, B.Cu at (115.9, 114.8)
- added D4: D, Diode_SMD:D_SOD-123, B.Cu at (134.9, 67.1)
- added D5: D, Diode_SMD:D_SOD-123, B.Cu at (134.9, 86.2)
- added D6: D, Diode_SMD:D_SOD-123, B.Cu at (134.9, 105.2)
- added D7: D, Diode_SMD:D_SOD-123, B.Cu at (153.9, 67.1)
- added D8: D, Diode_SMD:D_SOD-123, B.Cu at (154.0, 86.1)
- added D9: D, Diode_SMD:D_SOD-123, B.Cu at (154.0, 105.1)
- added R1: 806k, Resistor_SMD:R_0805_2012Metric, F.Cu at (153.0, 51.3)
- added R2: 2M, Resistor_SMD:R_0805_2012Metric, F.Cu at (153.0, 49.3)
- added SW1: Switch, ScottoKeebs_Hotswap:Hotswap_MX, F.Cu at (107.5, 77.1)
- added SW10: Switch, ScottoKeebs_Hotswap:Hotswap_MX, F.Cu at (145.6, 105.6)
- added SW11: Switch, ScottoKeebs_Hotswap:Hotswap_MX, F.Cu at (164.6, 77.2)
- added SW12: Switch, ScottoKeebs_Hotswap:Hotswap_MX, F.Cu at (164.6, 96.0)
- added SW13: Switch, ScottoKeebs_Hotswap:Hotswap_MX, F.Cu at (164.6, 115.3)
- added SW14: Switch, ScottoKeebs_Hotswap:Hotswap_MX, F.Cu at (183.6, 115.3)
- added SW15: Switch, ScottoKeebs_Hotswap:Hotswap_MX, F.Cu at (183.5, 77.2)
- added SW16: Switch, ScottoKeebs_Hotswap:Hotswap_MX, F.Cu at (183.6, 96.2)
- added SW17: Switch, ScottoKeebs_Hotswap:Hotswap_MX, F.Cu at (164.6, 134.3)
- added SW2: Switch, ScottoKeebs_Hotswap:Hotswap_MX, F.Cu at (107.6, 96.2)
- added SW3: Switch, ScottoKeebs_Hotswap:Hotswap_MX, F.Cu at (107.5, 115.3)
- added SW4: Switch, ScottoKeebs_Hotswap:Hotswap_MX, F.Cu at (126.5, 67.6)
- added SW5: Switch, ScottoKeebs_Hotswap:Hotswap_MX, F.Cu at (126.5, 86.7)
- added SW6: Switch, ScottoKeebs_Hotswap:Hotswap_MX, F.Cu at (126.5, 105.7)
- added SW7: EC11, Rotary Encoders:RotaryEncoder_Alps_EC11E-Switch_Vertical_H20mm, F.Cu at (175.9, 129.6)
- added SW8: Switch, ScottoKeebs_Hotswap:Hotswap_MX, F.Cu at (145.5, 67.6)
- added SW9: Switch, ScottoKeebs_Hotswap:Hotswap_MX, F.Cu at (145.6, 86.6)
- added TP1: GND, TestPoint:TestPoint_Pad_D2.0mm, B.Cu at (136.5, 55.1)
- added TP2: VBAT, TestPoint:TestPoint_Pad_D2.0mm, B.Cu at (139.7, 55.1)
- added U1: XIAO-nRF52840-SMD, Fixed Footprints:XIAO-nRF52840-SMD Fixed, F.Cu at (164.7, 57.0)
Routing:
- net /ROW2: track 0.00 -> 183.9 mm, vias 0 -> 5
- net /Right/ROW2: track 178.6 -> 0.00 mm, vias 5 -> 0
- net /ROW1: track 0.00 -> 163.7 mm, vias 0 -> 7
- net /Right/ROW1: track 163.3 -> 0.00 mm, vias 7 -> 0
- net Net-(C4-Pad1): track 148.6 -> 0.00 mm, vias 2 -> 0
- net /Right/ROW0: track 138.4 -> 0.00 mm, vias 7 -> 0
- net /COL1: track 0.00 -> 136.9 mm, vias 0 -> 1
- net /ROW0: track 0.00 -> 136.5 mm, vias 0 -> 7
- net Net-(C3-Pad2): track 124.6 -> 0.00 mm, vias 6 -> 0
- net /Right/COL0: track 111.9 -> 0.00 mm, vias 1 -> 0
- net /COL0: track 0.00 -> 111.8 mm, vias 0 -> 1
- net /SW: track 0.00 -> 100.4 mm
- net /R_Encoder_B: track 0.00 -> 95.4 mm
- net /R_Encoder_A: track 0.00 -> 93.8 mm
- net /Right/SW: track 92.3 -> 0.00 mm
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
Commit message: Add Separate Cads
Parts:
- moved D13 38.2 mm to (192.0, 76.6)
- moved SW14 38.1 mm to (184.1, 77.2)
- moved SW16 19.2 mm to (184.1, 115.4)
- moved D15 19.1 mm to (192.0, 114.8)
- moved SW15 19.1 mm to (184.1, 96.2)
- moved D14 19.0 mm to (191.9, 95.8)
- moved SW17 0.42 mm to (164.9, 134.6)
- moved SW12 0.37 mm to (164.9, 96.3)
- moved SW10 0.35 mm to (145.8, 105.9)
- moved SW13 0.32 mm to (164.9, 115.4)
- moved SW8 0.30 mm to (145.8, 67.6)
- moved SW11 0.26 mm to (164.9, 77.2)
- moved SW9 0.22 mm to (145.8, 86.7)
- moved SW6 0.22 mm to (126.6, 105.9)
- moved SW2 0.20 mm to (107.4, 96.2)
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Connections:
- SW17 pad 1: /COL1 -> /COL3
Routing:
- net /COL1: track 136.9 -> 80.7 mm
- net /ROW2: track 183.9 -> 167.6 mm
- net /ROW1: track 163.7 -> 156.9 mm, vias 7 -> 5
- net GND: track 0.00 -> 4.63 mm, vias 119 -> 52
- net Net-(D13-A): track 0.00 -> 3.96 mm
- net /COL3: track 73.0 -> 74.9 mm
- net /ROW3: track 82.7 -> 84.6 mm
- net /COL0: track 111.8 -> 113.5 mm
- net /R_Encoder_A: track 93.8 -> 92.3 mm
- net /ROW0: track 136.5 -> 135.9 mm
- net /COL2: track 60.7 -> 60.1 mm
- net /COL4: track 67.1 -> 66.7 mm, vias 1 -> 3
