File: Hardware/Right Split Keyboard.kicad_pcb (KiCad board)
At the start: 2 copper layers, 99.2 x 97.7 mm, 44 parts, among them CN1 1.0-2P WT, SW1 Switch, SW10 Switch, SW11 Switch, SW12 Switch, SW13 Switch, SW14 Switch, SW15 Switch, SW16 Switch, SW17 Switch, SW2 Switch, SW3 Switch, SW4 Switch, SW5 Switch, SW6 Switch, SW7 EC11, SW8 Switch, SW9 Switch, U1 XIAO-nRF52840-SMD

Commit message: Finally Final
Parts:
- added REF**: MountingHole_2.2mm_M2, MountingHole:MountingHole_2.2mm_M2, F.Cu at (179.8, 123.2)
- added REF**: MountingHole_2.2mm_M2, MountingHole:MountingHole_2.2mm_M2, F.Cu at (182.5, 56.8)
- added REF**: MountingHole_2.2mm_M2, MountingHole:MountingHole_2.2mm_M2, F.Cu at (105.8, 59.5)
- added REF**: MountingHole_2.2mm_M2, MountingHole:MountingHole_2.2mm_M2, F.Cu at (105.8, 139.5)
- added REF**: MountingHole_2.2mm_M2, MountingHole:MountingHole_2.2mm_M2, F.Cu at (147.2, 123.2)
- added REF**: MountingHole_2.2mm_M2, MountingHole:MountingHole_2.2mm_M2, F.Cu at (157.8, 52.0)
Routing:
- net Net-(C2-Pad1): track 93.4 -> 102.2 mm
- net /Left/ROW2: track 174.8 -> 181.4 mm
- net /Left/ROW0: track 123.7 -> 126.9 mm
- net /Left/ROW1: track 138.7 -> 141.9 mm
- net /Left/ROW3: track 128.7 -> 131.5 mm
- net /Left/VBAT: track 44.3 -> 42.2 mm
- net /Left/COL4: track 114.1 -> 113.5 mm
- net GND: vias 194 -> 147

Commit message: Plate fixes
Parts:
- removed C1, C2, C5: 10nF, Capacitor_SMD:C_0805_2012Metric
- removed CN1: 1.0-2P WT, lcsc:CONN-SMD_2P-P1.00_SHOU-HAN_1.0-2P-WT
- removed D1, D10, D11, D12, D13, D14, D15, D16, D2, D3, D4, D5, D6, D7, D8, D9: D, Diode_SMD:D_SOD-123
- removed R1: 806k, Resistor_SMD:R_0805_2012Metric
- removed R2: 2M, Resistor_SMD:R_0805_2012Metric
- removed R3, R4: 10k, Resistor_SMD:R_0805_2012Metric
- removed SW1, SW10, SW11, SW12, SW13, SW14, SW15, SW16, SW17, SW2, SW3, SW4, SW5, SW6, SW8, SW9: Switch, ScottoKeebs_Hotswap:Hotswap_MX_1.00u
- removed SW7: EC11, Rotary Encoders:RotaryEncoder_Alps_EC11E-Switch_Vertical_H20mm
- removed TP1: GND, TestPoint:TestPoint_Pad_D2.0mm
- removed TP2: VBAT, TestPoint:TestPoint_Pad_D2.0mm
- removed U1: XIAO-nRF52840-SMD, Fixed Footprints:XIAO-nRF52840-SMD Fixed
- added CN2: 1.0-2P WT, lcsc:CONN-SMD_2P-P1.00_SHOU-HAN_1.0-2P-WT, F.Cu at (150.4, 49.6)
- added D17: D, Diode_SMD:D_SOD-123, B.Cu at (124.4, 75.1)
- added D18: D, Diode_SMD:D_SOD-123, B.Cu at (124.4, 94.1)
- added D19: D, Diode_SMD:D_SOD-123, B.Cu at (124.3, 113.1)
- added D20: D, Diode_SMD:D_SOD-123, B.Cu at (143.3, 75.0)
- added D21: D, Diode_SMD:D_SOD-123, B.Cu at (143.3, 94.1)
- added D22: D, Diode_SMD:D_SOD-123, B.Cu at (143.3, 113.1)
- added D23: D, Diode_SMD:D_SOD-123, B.Cu at (162.3, 67.2)
- added D24: D, Diode_SMD:D_SOD-123, B.Cu at (162.3, 86.1)
- added D25: D, Diode_SMD:D_SOD-123, B.Cu at (162.4, 105.2)
- added D26: D, Diode_SMD:D_SOD-123, B.Cu at (181.3, 67.2)
- added D27: D, Diode_SMD:D_SOD-123, B.Cu at (181.4, 86.1)
- added D28: D, Diode_SMD:D_SOD-123, B.Cu at (181.3, 105.1)
- added D29: D, Diode_SMD:D_SOD-123, B.Cu at (200.4, 76.6)
- added D30: D, Diode_SMD:D_SOD-123, B.Cu at (200.4, 95.5)
- added D31: D, Diode_SMD:D_SOD-123, B.Cu at (200.4, 114.6)
- added D32: D, Diode_SMD:D_SOD-123, B.Cu at (143.3, 132.1)
- added R5: 806k, Resistor_SMD:R_0805_2012Metric, F.Cu at (121.6, 50.0)
- added R6: 2M, Resistor_SMD:R_0805_2012Metric, F.Cu at (121.6, 48.0)
- added SW18: Switch, ScottoKeebs_Hotswap:Hotswap_MX_1.00u, F.Cu at (115.9, 75.6)
- added SW19: Switch, ScottoKeebs_Hotswap:Hotswap_MX_1.00u, F.Cu at (116.0, 94.6)
- added SW20: Switch, ScottoKeebs_Hotswap:Hotswap_MX_1.00u, F.Cu at (115.9, 113.6)
- added SW21: Switch, ScottoKeebs_Hotswap:Hotswap_MX_1.00u, F.Cu at (134.9, 75.6)
- added SW22: Switch, ScottoKeebs_Hotswap:Hotswap_MX_1.00u, F.Cu at (134.9, 94.6)
- added SW23: Switch, ScottoKeebs_Hotswap:Hotswap_MX_1.00u, F.Cu at (134.9, 113.6)
- added SW24: EC11, Rotary Encoders:RotaryEncoder_Alps_EC11E-Switch_Vertical_H20mm, F.Cu at (109.5, 127.8)
- added SW25: Switch, ScottoKeebs_Hotswap:Hotswap_MX_1.00u, F.Cu at (153.9, 67.7)
- added SW26: Switch, ScottoKeebs_Hotswap:Hotswap_MX_1.00u, F.Cu at (153.9, 86.6)
- added SW27: Switch, ScottoKeebs_Hotswap:Hotswap_MX_1.00u, F.Cu at (153.9, 105.7)
- added SW28: Switch, ScottoKeebs_Hotswap:Hotswap_MX_1.00u, F.Cu at (172.9, 67.7)
- added SW29: Switch, ScottoKeebs_Hotswap:Hotswap_MX_1.00u, F.Cu at (173.0, 86.6)
- added SW30: Switch, ScottoKeebs_Hotswap:Hotswap_MX_1.00u, F.Cu at (172.9, 105.6)
- added SW31: Switch, ScottoKeebs_Hotswap:Hotswap_MX_1.00u, F.Cu at (191.9, 77.1)
- added SW32: Switch, ScottoKeebs_Hotswap:Hotswap_MX_1.00u, F.Cu at (191.9, 96.1)
- added SW33: Switch, ScottoKeebs_Hotswap:Hotswap_MX_1.00u, F.Cu at (191.9, 115.1)
- added SW34: Switch, ScottoKeebs_Hotswap:Hotswap_MX_1.00u, F.Cu at (134.8, 132.6)
- added TP3: GND, TestPoint:TestPoint_Pad_D2.0mm, B.Cu at (148.8, 53.5)
- added TP4: VBAT, TestPoint:TestPoint_Pad_D2.0mm, B.Cu at (144.8, 53.5)
- added U2: XIAO-nRF52840-SMD, Fixed Footprints:XIAO-nRF52840-SMD Fixed, F.Cu at (133.4, 55.6)
Routing:
- net /Left/ROW2: track 181.4 -> 0.00 mm, vias 6 -> 0
- net /ROW2: track 0.00 -> 174.9 mm, vias 0 -> 6
- net /Left/ROW1: track 141.9 -> 0.00 mm, vias 6 -> 0
- net /ROW1: track 0.00 -> 141.8 mm, vias 0 -> 6
- net /Left/ROW3: track 131.5 -> 0.00 mm, vias 1 -> 0
- net /ROW3: track 0.00 -> 130.4 mm, vias 0 -> 1
- net /ROW0: track 0.00 -> 127.0 mm, vias 0 -> 5
- net /Left/ROW0: track 126.9 -> 0.00 mm, vias 5 -> 0
- net /COL4: track 0.00 -> 114.9 mm, vias 0 -> 1
- net /Left/COL4: track 113.5 -> 0.00 mm, vias 1 -> 0
- net /R_Encoder_B: track 0.00 -> 112.6 mm, vias 0 -> 2
- net Net-(C2-Pad1): track 102.2 -> 0.00 mm
- net /R_Encoder_A: track 0.00 -> 101.7 mm, vias 0 -> 1
- net Net-(C1-Pad2): track 92.7 -> 0.00 mm, vias 1 -> 0
- net /Left/SW: track 86.7 -> 0.00 mm, vias 1 -> 0
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
Commit message: Add Separate Cads
Parts:
- moved SW30 0.10 mm to (172.9, 105.7)
- moved U2 0.10 mm to (133.4, 55.7)
Routing:
- net GND: track 0.00 -> 2.55 mm, vias 8 -> 40
- net /VBAT: track 47.2 -> 46.3 mm
